File: hardware/maciot-board.sch (KiCad schematic (older format))
At the start: 72 parts, among them P1 Power, P101 USB_OTG, P102 TST, P103 TST, P104 TST, P105 TST, P106 TST, P107 TST, P108 TST, P109 TST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

Commit message: added cap pad
Parts:
- removed R?: 10k, w_smd_resistors:r_0805, symbol R
- added C?: 10nf, w_smd_cap:c_0805, symbol C
- added R?: 10k, w_smd_resistors:r_0805, symbol R
- added R? (x2): 0, w_smd_resistors:r_0805, symbol R
- added R?: R, symbol device:R
- added SW1: CPad 1, symbol TEST_1P
- D1, D102, D103, D104, D105: symbol LED-RESCUE-maciot-board -> maciot-board-rescue:LED-RESCUE-maciot-board
- P101: symbol USB_OTG-RESCUE-maciot-board -> maciot-board-rescue:USB_OTG-RESCUE-maciot-board
- U101: symbol LM1117IMPX-ADJ -> lm1117:LM1117IMPX-ADJ
- U102: symbol CP2102 -> CP2102:CP2102
- U103: symbol ESP32-WROOM -> espressif-xess:ESP32-WROOM
Connections:
- wire segments 204 -> 250
Other:
- moved on the sheet: C101, C102, R103, R104, R105, R106, R107, SW101, SW102
